Commit message: added ros2_control ackermann steering controller

File: description/robot.urdf.xacro (robot description, xacro)
@@ -2,4 +2,5 @@
 <robot xmlns:xacro="http://www.ros.org/wiki/xacro"  name="robot">
     <xacro:include filename="robot_core.xacro" />
- <xacro:include filename="gazebo_control.xacro" />
+ <xacro:include filename="ros2_control.xacro" />
+    <xacro:include filename="gazebo_control.xacro" />
 </robot>

File: description/robot_core.xacro (robot description, xacro)
@@ -153,5 +153,5 @@
             <origin xyz="-8.09391e-17 7.65875e-18 0.17" rpy="1.5708 0 0"/>
             <geometry>
-                    <mesh filename="file:///home/jay/ros2_ws/src/articubot_one/description/assets/wheel.stl"/>
+                    <sphere radius="0.2"/>
                  <!--  <box size="0.3 0.3 0.15"/> -->
             </geometry>
@@ -184,5 +184,5 @@
             <origin xyz="-1.59877e-17 7.65404e-18 0.17" rpy="1.5708 0 0"/>
             <geometry>
-                    <mesh filename="file:///home/jay/ros2_ws/src/articubot_one/description/assets/wheel.stl"/>
+                     <sphere radius="0.2"/>
                  <!--  <box size="0.3 0.3 0.15"/> -->
             </geometry>
@@ -227,5 +227,5 @@
         <material>Gazebo/Black</material>
     </gazebo>
-    <joint name="FRwheel" type="continuous">
+    <joint name="FRWheel" type="continuous">
         <origin xyz="0.10836 0 0.09" rpy="1.5708 0 -1.5708"/>
         <parent link="front_right_wheel_hub"/>
@@ -246,5 +246,6 @@
             <origin xyz="2.22045e-16 0 0.17" rpy="1.5708 0 1.5708"/>
             <geometry>
-                    <mesh filename="file:///home/jay/ros2_ws/src/articubot_one/description/assets/wheel.stl"/>
+                   <!-- <mesh filename="file:///home/jay/ros2_ws/src/articubot_one/description/assets/wheel.stl"/>      -->
+                    <sphere radius="0.2"/>
                  <!--  <box size="0.3 0.3 0.15"/> -->
             </geometry>
@@ -308,5 +309,5 @@
         <origin xyz="0 0 0.17" rpy="1.5708 0 0"/>
         <geometry>
-                    <mesh filename="file:///home/jay/ros2_ws/src/articubot_one/description/assets/wheel.stl"/>
+                     <sphere radius="0.2"/>
                  <!--  <box size="0.3 0.3 0.15"/> -->
         </geometry>
@@ -319,4 +320,5 @@
         <material>Gazebo/Grey</material>
     </gazebo>
+<!--
         <gazebo>
            <plugin
@@ -335,5 +337,4 @@
                 <max_velocity>10</max_velocity>
                 <max_acceleration>5.0</max_acceleration>
-                <!-- REVERSE DONUT SIM <max_jerk>10.0</max_jerk> -->
                  <odom_topic>/model/my_robot/odometry</odom_topic>
               <tf_topic>/model/my_robot/tf</tf_topic>
@@ -348,12 +349,4 @@
           <static_update_frequency>50</static_update_frequency>
         </plugin>
-   <!--
-       <plugin name="ignition::gazebo::systems::OdometryPublisher"
-        filename="libignition-gazebo6-odometry-publisher-system.so">
-  <odom_frame>odom</odom_frame>
-  <robot_base_frame>base_link</robot_base_frame>
-  -->
-      <!-- ign topic -t "/model/my_robot/cmd_vel" -m ignition.msgs.Twist -p "linear: {x: 5}, angular: {z: -5}"
- -->
       <plugin filename="libignition-gazebo-joint-state-publisher-system.so"
         name="ignition::gazebo::systems::JointStatePublisher">
@@ -362,3 +355,4 @@
       </plugin>
       </gazebo>
+-->
 </robot>

Commit message: added depth camera simulation into gazebo and reading into ROS2/RVIZ2

File: description/robot.urdf.xacro (robot description, xacro)
@@ -2,5 +2,8 @@
 <robot xmlns:xacro="http://www.ros.org/wiki/xacro"  name="robot">
     <xacro:include filename="robot_core.xacro" />
- <xacro:include filename="ros2_control.xacro" />
-    <xacro:include filename="gazebo_control.xacro" />
+    <xacro:include filename="ros2_control.xacro" />
+    <xacro:include filename="gazebo_control.xacro"/>
+   <!-- <xacro:include filename="camera.xacro" /> -->
+    <!--<xacro:include filename="depthcamera.xacro" /> -->
+     <xacro:include filename="rgbdcamera.xacro" />
 </robot>

File: description/robot_core.xacro (robot description, xacro)
@@ -27,5 +27,5 @@
     <link name="chassis">
         <visual>
-            <origin xyz="2.1706 -0.00985747 0.0751" rpy="3.14159 0 1.5708"/>
+            <origin xyz="2.2924 -0.00985747 0.0751" rpy="3.14159 0 1.5708"/>
             <geometry>
                   <mesh filename="file:///home/jay/ros2_ws/src/articubot_one/description/assets/chassis.stl"/>
@@ -47,5 +47,5 @@
      <!-- Part rear_suspension -->
     <visual>
-      <origin xyz="-0.17247 -0.28192 0.105" rpy="3.14159 5.47382e-48 -0.0851102"/>
+      <origin xyz="-0.170629 -0.28192 0.105" rpy="3.14159 5.47382e-48 -0.0851102"/>
       <geometry>
         <mesh filename="file:///home/jay/ros2_ws/src/articubot_one/description/assets/rear_suspension.stl"/>
@@ -54,5 +54,5 @@
     </visual>
     <collision>
-      <origin xyz="-0.17247 -0.28192 0.105" rpy="3.14159 5.47382e-48 -0.0851102"/>
+      <origin xyz="-0.170629 -0.28192 0.105" rpy="3.14159 5.47382e-48 -0.0851102"/>
       <geometry>
         <mesh filename="file:///home/jay/ros2_ws/src/articubot_one/description/assets/rear_suspension.stl"/>
@@ -196,4 +196,5 @@
     </gazebo>
     <!-- FRONT RIGHT STEERING ASSEMBLY -->
+    <!-- FRONT RIGHT STEERING ASSEMBLY -->
     <joint name="RSteer" type="revolute">
         <origin xyz="1.739 -0.584139 0.075" rpy="-3.14159 0 -1.5708"/>
@@ -232,5 +233,6 @@
         <child link="front_right_wheel"/>
         <axis xyz="0 0 1"/>
-        <limit effort="0.0" velocity="100"/>
+        <limit effort="50" velocity="100"/>
+        <dynamics damping="0.0" friction="0.0"/>
     </joint>
     <link name="front_right_wheel">
@@ -295,5 +297,6 @@
         <child link="front_left_wheel"/>
         <axis xyz="0 0 1"/>
-        <limit effort="0.0" velocity="100"/>
+        <limit effort="50" velocity="100"/>
+        <dynamics damping="0.0" friction="0.0"/>
     </joint>
     <link name="front_left_wheel">

File: description/ros2_control.xacro (robot description, xacro)
@@ -6,30 +6,31 @@
     </hardware>
   <!-- front steering -->
-    <joint name="LSteer">
-      <command_interface name="position"/>
-      <state_interface   name="position"/>
-    </joint>
-    <joint name="RSteer">
-      <command_interface name="position"/>
-      <state_interface   name="position"/>
-    </joint>
-    <!-- rear drive -->
-    <joint name="RLMotor">
-      <command_interface name="velocity"/>
-      <state_interface   name="velocity"/>
-      <state_interface   name="position"/>
-    </joint>
-    <joint name="RRMotor">
-      <command_interface name="velocity"/>
-      <state_interface   name="velocity"/>
-      <state_interface   name="position"/>
-    </joint>
-    <joint name="FLWheel">
-      <state_interface   name="position"/>
-    </joint>
-    <joint name="FRWheel">
-      <state_interface   name="position"/>
-    </joint>
-  </ros2_control>
+  <joint name="LSteer">
+    <command_interface name="position"/>
+    <state_interface   name="position"/>
+  </joint>
+  <joint name="RSteer">
+    <command_interface name="position"/>
+    <state_interface   name="position"/>
+  </joint>
+  <!-- rear drive -->
+  <joint name="RLMotor">
+    <command_interface name="velocity"/>
+    <state_interface   name="velocity"/>
+    <state_interface   name="position"/>
+  </joint>
+  <joint name="RRMotor">
+    <command_interface name="velocity"/>
+    <state_interface   name="velocity"/>
+    <state_interface   name="position"/>
+  </joint>
+  <!-- front wheels (braking via effort command) -->
+  <joint name="FLWheel">
+    <state_interface   name="position"/>
+  </joint>
+  <joint name="FRWheel">
+    <state_interface   name="position"/>
+  </joint>
+</ros2_control>
   <gazebo>
     <plugin filename="gz_ros2_control-system" name="gz_ros2_control::GazeboSimROS2ControlPlugin">

Commit message: working localisation using SLAM Toolbox, with fusion between imu and wheel odom

File: description/robot.urdf.xacro (robot description, xacro)
@@ -6,4 +6,6 @@
    <!-- <xacro:include filename="camera.xacro" /> -->
     <!--<xacro:include filename="depthcamera.xacro" /> -->
-     <xacro:include filename="rgbdcamera.xacro" />
+   <xacro:include filename="rgbdcamera.xacro" />
+   <xacro:include filename="sensors.xacro" />
+   <xacro:include filename="lidar.xacro" />
 </robot>

File: description/robot_core.xacro (robot description, xacro)
@@ -18,4 +18,11 @@
     <link name="base_link">
       <!-- You can add visual, collision, and inertial info here -->
+    </link>
+    <joint name="base_footprint_joint" type="fixed">
+        <parent link="base_link"/>
+        <child link="base_footprint"/>
+        <origin xyz="0 0 0" rpy="0 0 0"/>
+    </joint>
+    <link name="base_footprint">
     </link>
     <!-- Fixed joint connecting base_link to chassis -->
