Commit message: corrected naming of project

File: description/robot_core.xacro (robot description, xacro)
@@ -30,5 +30,5 @@
       <parent link="base_link"/>
       <child link="chassis"/>
-      <origin xyz="0 0 0.2028" rpy="0 0 0"/>
+      <origin xyz="-0.9 0 0.2028" rpy="0 0 0"/>
     </joint>
     <link name="chassis">
@@ -36,6 +36,6 @@
             <origin xyz="2.2924 -0.00985747 0.0751" rpy="3.14159 0 1.5708"/>
             <geometry>
-                  <mesh filename="file:///home/jay/ros2_ws/src/articubot_one/description/assets/chassis.stl"/>
-                 <!-- <mesh filename="package://articubot_one/description/assets/chassis.stl"/> -->
+                  <mesh filename="file:///home/jay/ros2_ws/src/avone/description/assets/chassis.stl"/>
+                 <!-- <mesh filename="package://avone/description/assets/chassis.stl"/> -->
                  <!--  <box size="0.3 0.3 0.15"/> -->
             </geometry>
@@ -45,5 +45,5 @@
             <origin xyz="2.2924 -0.00985747 0.0751" rpy="3.14159 0 1.5708"/>
             <geometry>
-                    <mesh filename="file:///home/jay/ros2_ws/src/articubot_one/description/assets/chassis.stl"/>
+                    <mesh filename="file:///home/jay/ros2_ws/src/avone/description/assets/chassis.stl"/>
                  <!--  <box size="0.3 0.3 0.15"/> -->
             </geometry>
@@ -56,5 +56,5 @@
       <origin xyz="-0.170629 -0.28192 0.105" rpy="3.14159 5.47382e-48 -0.0851102"/>
       <geometry>
-        <mesh filename="file:///home/jay/ros2_ws/src/articubot_one/description/assets/rear_suspension.stl"/>
+        <mesh filename="file:///home/jay/ros2_ws/src/avone/description/assets/rear_suspension.stl"/>
       </geometry>
       <material name="blue"/>
@@ -63,5 +63,5 @@
       <origin xyz="-0.170629 -0.28192 0.105" rpy="3.14159 5.47382e-48 -0.0851102"/>
       <geometry>
-        <mesh filename="file:///home/jay/ros2_ws/src/articubot_one/description/assets/rear_suspension.stl"/>
+        <mesh filename="file:///home/jay/ros2_ws/src/avone/description/assets/rear_suspension.stl"/>
       </geometry>
     </collision>
@@ -70,5 +70,5 @@
       <origin xyz="0.189017 0.312761 0.105" rpy="-3.14159 2.33363e-61 -3.05648"/>
       <geometry>
-        <mesh filename="file:///home/jay/ros2_ws/src/articubot_one/description/assets/rear_suspension.stl"/>
+        <mesh filename="file:///home/jay/ros2_ws/src/avone/description/assets/rear_suspension.stl"/>
       </geometry>
       <material name="blue"/>
@@ -77,5 +77,5 @@
       <origin xyz="0.189017 0.312761 0.105" rpy="-3.14159 2.33363e-61 -3.05648"/>
       <geometry>
-        <mesh filename="file:///home/jay/ros2_ws/src/articubot_one/description/assets/rear_suspension.stl"/>
+        <mesh filename="file:///home/jay/ros2_ws/src/avone/description/assets/rear_suspension.stl"/>
       </geometry>
     </collision>
@@ -84,5 +84,5 @@
       <origin xyz="1.6032 0.2935 0.075" rpy="3.14159 -1.54112e-16 1.5708"/>
       <geometry>
-        <mesh filename="file:///home/jay/ros2_ws/src/articubot_one/description/assets/front_suspension.stl"/>
+        <mesh filename="file:///home/jay/ros2_ws/src/avone/description/assets/front_suspension.stl"/>
       </geometry>
       <material name="blue"/>
@@ -91,5 +91,5 @@
       <origin xyz="1.6032 0.2935 0.075" rpy="3.14159 -1.54112e-16 1.5708"/>
       <geometry>
-        <mesh filename="file:///home/jay/ros2_ws/src/articubot_one/description/assets/front_suspension.stl"/>
+        <mesh filename="file:///home/jay/ros2_ws/src/avone/description/assets/front_suspension.stl"/>
       </geometry>
     </collision>
@@ -98,5 +98,5 @@
       <origin xyz="1.8748 -0.2935 0.075" rpy="-3.14159 1.54112e-16 -1.5708"/>
       <geometry>
-        <mesh filename="file:///home/jay/ros2_ws/src/articubot_one/description/assets/front_suspension.stl"/>
+        <mesh filename="file:///home/jay/ros2_ws/src/avone/description/assets/front_suspension.stl"/>
       </geometry>
       <material name="blue"/>
@@ -105,5 +105,5 @@
       <origin xyz="1.8748 -0.2935 0.075" rpy="-3.14159 1.54112e-16 -1.5708"/>
       <geometry>
-        <mesh filename="file:///home/jay/ros2_ws/src/articubot_one/description/assets/front_suspension.stl"/>
+        <mesh filename="file:///home/jay/ros2_ws/src/avone/description/assets/front_suspension.stl"/>
       </geometry>
     </collision>
@@ -112,5 +112,5 @@
       <origin xyz="-0.181377 0.297001 -0.105" rpy="6.30462e-15 0 -6.18615e-05"/>
       <geometry>
-        <mesh filename="file:///home/jay/ros2_ws/src/articubot_one/description/assets/rear_wheel_hub.stl"/>
+        <mesh filename="file:///home/jay/ros2_ws/src/avone/description/assets/rear_wheel_hub.stl"/>
       </geometry>
       <material name="white"/>
@@ -119,5 +119,5 @@
       <origin xyz="-0.181377 0.297001 -0.105" rpy="6.30462e-15 0 -6.18615e-05"/>
       <geometry>
-        <mesh filename="file:///home/jay/ros2_ws/src/articubot_one/description/assets/rear_wheel_hub.stl"/>
+        <mesh filename="file:///home/jay/ros2_ws/src/avone/description/assets/rear_wheel_hub.stl"/>
       </geometry>
     </collision>
@@ -126,5 +126,5 @@
       <origin xyz="0.181423 -0.296978 -0.105" rpy="3.10966e-15 7.00787e-15 -3.14153"/>
       <geometry>
-        <mesh filename="file:///home/jay/ros2_ws/src/articubot_one/description/assets/rear_wheel_hub.stl"/>
+        <mesh filename="file:///home/jay/ros2_ws/src/avone/description/assets/rear_wheel_hub.stl"/>
       </geometry>
       <material name="white"/>
@@ -133,5 +133,5 @@
       <origin xyz="0.181423 -0.296978 -0.105" rpy="3.10966e-15 7.00787e-15 -3.14153"/>
       <geometry>
-        <mesh filename="file:///home/jay/ros2_ws/src/articubot_one/description/assets/rear_wheel_hub.stl"/>
+        <mesh filename="file:///home/jay/ros2_ws/src/avone/description/assets/rear_wheel_hub.stl"/>
       </geometry>
     </collision>
@@ -152,5 +152,5 @@
             <origin xyz="-8.09391e-17 7.65875e-18 0.17" rpy="1.5708 0 0"/>
             <geometry>
-                    <mesh filename="file:///home/jay/ros2_ws/src/articubot_one/description/assets/wheel.stl"/>
+                    <mesh filename="file:///home/jay/ros2_ws/src/avone/description/assets/wheel.stl"/>
                  <!--  <box size="0.3 0.3 0.15"/> -->
             </geometry>
@@ -183,5 +183,5 @@
             <origin xyz="-1.59877e-17 7.65404e-18 0.17" rpy="1.5708 0 0"/>
             <geometry>
-                    <mesh filename="file:///home/jay/ros2_ws/src/articubot_one/description/assets/wheel.stl"/>
+                    <mesh filename="file:///home/jay/ros2_ws/src/avone/description/assets/wheel.stl"/>
                  <!--  <box size="0.3 0.3 0.15"/> -->
             </geometry>
@@ -216,5 +216,5 @@
             <origin xyz="-0.290639 0.1358 0.18" rpy="-3.14159 0 0"/>
             <geometry>
-                    <mesh filename="file:///home/jay/ros2_ws/src/articubot_one/description/assets/front_wheel_hub.stl"/>
+                    <mesh filename="file:///home/jay/ros2_ws/src/avone/description/assets/front_wheel_hub.stl"/>
                  <!--  <box size="0.3 0.3 0.15"/> -->
             </geometry>
@@ -224,5 +224,5 @@
             <origin xyz="-0.290639 0.1358 0.18" rpy="-3.14159 0 0"/>
             <geometry>
-                    <mesh filename="file:///home/jay/ros2_ws/src/articubot_one/description/assets/front_wheel_hub.stl"/>
+                    <mesh filename="file:///home/jay/ros2_ws/src/avone/description/assets/front_wheel_hub.stl"/>
                  <!--  <box size="0.3 0.3 0.15"/> -->
             </geometry>
@@ -247,5 +247,5 @@
             <origin xyz="2.22045e-16 0 0.17" rpy="1.5708 0 1.5708"/>
             <geometry>
-                    <mesh filename="file:///home/jay/ros2_ws/src/articubot_one/description/assets/wheel.stl"/>
+                    <mesh filename="file:///home/jay/ros2_ws/src/avone/description/assets/wheel.stl"/>
                  <!--  <box size="0.3 0.3 0.15"/> -->
             </geometry>
@@ -255,5 +255,5 @@
             <origin xyz="2.22045e-16 0 0.17" rpy="1.5708 0 1.5708"/>
             <geometry>
-                   <!-- <mesh filename="file:///home/jay/ros2_ws/src/articubot_one/description/assets/wheel.stl"/>      -->
+                   <!-- <mesh filename="file:///home/jay/ros2_ws/src/avone/description/assets/wheel.stl"/>      -->
                     <sphere radius="0.2"/>
                  <!--  <box size="0.3 0.3 0.15"/> -->
@@ -280,5 +280,5 @@
         <origin xyz="-0.290639 0.1358 0.18" rpy="3.14159 0 0"/>
         <geometry>
-                    <mesh filename="file:///home/jay/ros2_ws/src/articubot_one/description/assets/front_wheel_hub.stl"/>
+                    <mesh filename="file:///home/jay/ros2_ws/src/avone/description/assets/front_wheel_hub.stl"/>
                  <!--  <box size="0.3 0.3 0.15"/> -->
         </geometry>
@@ -288,5 +288,5 @@
         <origin xyz="-0.290639 0.1358 0.18" rpy="3.14159 0 0"/>
         <geometry>
-                    <mesh filename="file:///home/jay/ros2_ws/src/articubot_one/description/assets/front_wheel_hub.stl"/>
+                    <mesh filename="file:///home/jay/ros2_ws/src/avone/description/assets/front_wheel_hub.stl"/>
                  <!--  <box size="0.3 0.3 0.15"/> -->
         </geometry>
@@ -311,5 +311,5 @@
         <origin xyz="0 0 0.17" rpy="1.5708 0 0"/>
         <geometry>
-                    <mesh filename="file:///home/jay/ros2_ws/src/articubot_one/description/assets/wheel.stl"/>
+                    <mesh filename="file:///home/jay/ros2_ws/src/avone/description/assets/wheel.stl"/>
                  <!--  <box size="0.3 0.3 0.15"/> -->
         </geometry>

File: description/ros2_control.xacro (robot description, xacro)
@@ -37,5 +37,5 @@
      <robot_param>robot_description</robot_param>
         <robot_param_node>robot_state_publisher</robot_param_node>
-      <parameters>$(find articubot_one)/config/ackermann_drive_controller.yaml</parameters>
+      <parameters>$(find avone)/config/ackermann_drive_controller.yaml</parameters>
     </plugin>
   </gazebo>
